File: Basic_circuits/VoltageDivider.sch (EAGLE design)
At the start: 2 parts

Commit message: Added pdf versions
Parts:
- added R3, R4, R5: 10k, rcl:R-EU_VTA52
Connections:
- new net OUT1: R3.2, R4.1
- new net OUT2: R3.1, R5.2
- net +5V: now also R4.2
- net GND: now also R5.1
Other:
- note added: "1/2 VIN"
- note added: "1/3 VIN"
- note added: "2/3 VIN"
- moved on the sheet: R1, R2
